File: pcb/Xing Signals XIAO.kicad_sch (KiCad schematic)
At the start: 48 parts, among them J1 Barrel_Jack_Switch, J10 Signals, J2 DCC IN, J3 Signals, J4 Signal Gate 1, J5 Signal Gate 2, J6 Conn_01x07_Pin, J7 Sensor Power, J8 Screw_Terminal_01x04, J9 Conn_01x07_Pin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

Commit message: Version 1.1 of the PCB
Parts:
- removed J4: Signal Gate 1, Connector_PinHeader_2.54mm:PinHeader_1x03_P2.54mm_Vertical, symbol Connector:Conn_01x03_Pin
- removed J5: Signal Gate 2, Connector_PinHeader_2.54mm:PinHeader_1x03_P2.54mm_Vertical, symbol Connector:Conn_01x03_Pin
- removed R1: 100ohm, Resistor_SMD:R_1206_3216Metric, symbol Device:R_US
- removed R16, R17: 100, Resistor_SMD:R_0402_1005Metric, symbol Device:R_Small_US
- added J4: Conn_02x03_Top_Bottom, Connector_PinHeader_2.54mm:PinHeader_2x03_P2.54mm_Vertical, symbol Connector_Generic:Conn_02x03_Top_Bottom
- added R1, R18, R19, R20: 100, Resistor_SMD:R_0402_1005Metric, symbol Device:R_Small_US
- R2: value 100ohm -> 1k; Comment 250mW Thick Film Resistors ±100ppm/℃ ±1% 100Ω 1206 Chip Res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 -> 250mW Thick Film Resistors 200V ±1% 1000Ω 1206 Chip Resisto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; LCSC C17901 -> C4410
- R3: value 200 -> 1k; Field5 62.5mW Thick Film Resistors ±100ppm/℃ ±1% 200Ω 0402 Chip Re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 -> 250mW Thick Film Resistors ±100ppm/℃ ±1% 300Ω 1206 Chip Res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; LCSC C25087 -> C17887
Connections:
- net +3V3: now also Q4.3 (C), Q5.3 (C), Q6.3 (C), Q7.3 (C), J4.3 (Pin_3), J4.4 (Pin_4)
- net GATE1: now also J4.6 (Pin_6)
- net GATE2: now also J4.5 (Pin_5)
- net GND: now also Q2.2 (E), Q3.2 (E), J4.1 (Pin_1), J4.2 (Pin_2), R1.1, R18.1, R19.1, R20.1; no longer D1.1 (K), D2.1 (K), D3.1 (K), D4.1 (K), D6.1 (K), D7.1 (K)
- net at D7.2 (A): now also D6.2 (A), J3.2 (Pin_2), R2.2
- net at J3.3 (Pin_3), Q3.3 (C): now also D7.1 (K)
- net at J3.1 (Pin_1), Q2.3 (C): now also D6.1 (K)
- new net: D1.1 (K), R19.2
- new net: D2.1 (K), R18.2
- new net: D4.1 (K), R20.2
- new net: D3.1 (K), R1.2
Other:
- moved on the sheet: D6, D7, Q2, Q3, R4, R5

Commit message: Fixes to Version 1.1
* Trace fixups
* Components moved to better fit
* Move the sensor screw terminals next to each other
* Cleaned up the transistor layout for the sensor LED indicators
* Servo pins are now 2x3
Parts:
- D5: value White -> Green; footprint LED_SMD:LED_0603_1608Metric -> LED_SMD:LED_0805_2012Metric; LCSC C2290 -> C2297
Changed lines of the file:
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@@
       (effects (font (size 1.27 1.27)) (justify right))
     )
-    (property "Value" "White" (at 212.09 51.1175 90)
+    (property "Value" "Green" (at 212.09 51.1175 90)
       (effects (font (size 1.27 1.27)) (justify right))
     )
-    (property "Footprint" "LED_SMD:LED_0603_1608Metric" (at 208.28 48.26 0)
+    (property "Footprint" "LED_SMD:LED_0805_2012Metric" (at 208.28 48.26 0)
       (effects (font (size 1.27 1.27)) hide)
     )
@@
       (effects (font (size 1.27 1.27)) hide)
     )
-    (property "LCSC" "C2290" (at 208.28 48.26 90)
+    (property "LCSC" "C2297" (at 208.28 48.26 90)
       (effects (font (size 1.27 1.27)) hide)
     )
-    (property "Description" "White 0603 Light Emitting Diodes (LED) ROHS" (at 208.28 48.26 90)
+    (property "Description" "Emerald 0805 Light Emitting Diodes (LED) ROHS" (at 208.28 48.26 90)
       (effects (font (size 1.27 1.27)) hide)
     )

Commit message: More fixes, ordered V1.1
* Added C3 to buffer the Servo current draw
* More fixes for traces
* Fixed TP2 to be VIN, not +12V
Parts:
- added C3: 47uf, Capacitor_SMD:C_0805_2012Metric, symbol Device:C_Small
- R3: LCSC C17887 -> C105637
- TP2: value +12V -> VIN
Connections:
- net +3V3: now also C3.1
- net GND: now also C3.2
Changed lines of the file:
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@@
   (junction (at 48.26 143.51) (diameter 0) (color 0 0 0 0)
   )
+  (junction (at 111.76 36.83) (diameter 0) (color 0 0 0 0)
+  )
   (junction (at 162.56 132.08) (diameter 0) (color 0 0 0 0)
   )
@@
   )
   (junction (at 173.99 41.91) (diameter 0) (color 0 0 0 0)
+  )
+  (junction (at 101.6 63.5) (diameter 0) (color 0 0 0 0)
   )
   (junction (at 194.31 41.91) (diameter 0) (color 0 0 0 0)
@@
     (stroke (width 0) (type default))
   )
+  (wire (pts (xy 111.76 36.83) (xy 111.76 31.75))
+    (stroke (width 0) (type default))
+  )
   (wire (pts (xy 118.11 137.16) (xy 118.11 158.75))
     (stroke (width 0) (type default))
@@
     (stroke (width 0) (type default))
   )
+  (wire (pts (xy 124.46 36.83) (xy 124.46 63.5))
+    (stroke (width 0) (type default))
+  )
   (wire (pts (xy 224.79 38.1) (xy 224.79 40.64))
     (stroke (width 0) (type default))
@@
     (stroke (width 0) (type default))
   )
+  (wire (pts (xy 116.84 36.83) (xy 124.46 36.83))
+    (stroke (width 0) (type default))
+  )
   (wire (pts (xy 242.57 129.54) (xy 242.57 132.08))
     (stroke (width 0) (type default))
@@
     (stroke (width 0) (type default))
   )
+  (wire (pts (xy 101.6 63.5) (xy 101.6 64.77))
+    (stroke (width 0) (type default))
+  )
   (wire (pts (xy 254 87.63) (xy 254 92.71))
     (stroke (width 0) (type default))
@@
     (stroke (width 0) (type default))
   )
-  (wire (pts (xy 111.76 43.18) (xy 111.76 31.75))
+  (wire (pts (xy 111.76 43.18) (xy 111.76 36.83))
     (stroke (width 0) (type default))
   )
@@
     (stroke (width 0) (type default))
   )
+  (wire (pts (xy 124.46 63.5) (xy 101.6 63.5))
+    (stroke (width 0) (type default))
+  )
   (wire (pts (xy 247.65 144.78) (xy 247.65 156.21))
     (stroke (width 0) (type default))
@@
     (stroke (width 0) (type default))
   )
-  (wire (pts (xy 101.6 48.26) (xy 101.6 64.77))
+  (wire (pts (xy 101.6 48.26) (xy 101.6 63.5))
     (stroke (width 0) (type default))
   )
@@
       (effects (font (size 1.27 1.27)) hide)
     )
-    (property "LCSC" "C17887" (at 205.74 41.91 90)
+    (property "LCSC" "C105637" (at 205.74 41.91 90)
       (effects (font (size 1.27 1.27)) hide)
     )
@@
     )
   )
+  (symbol (lib_id "Device:C_Small") (at 114.3 36.83 90) (unit 1)
+    (in_bom yes) (on_board yes) (dnp no) (fields_autoplaced)
+    (property "Reference" "C3" (at 114.3063 30.48 90)
+      (effects (font (size 1.27 1.27)))
+    )
+    (property "Value" "47uf" (at 114.3063 33.02 90)
+      (effects (font (size 1.27 1.27)))
+    )
+    (property "Footprint" "Capacitor_SMD:C_0805_2012Metric" (at 114.3 36.83 0)
+      (effects (font (size 1.27 1.27)) hide)
+    )
+    (property "Datasheet" "~" (at 114.3 36.83 0)
+      (effects (font (size 1.27 1.27)) hide)
+    )
+    (property "LCSC" "C16780" (at 114.3 36.83 90)
+      (effects (font (size 1.27 1.27)) hide)
+    )
+    (property "Description" "6.3V 47uF X5R ±20% 0805 Multilayer Ceramic Capacitors MLCC - SMD/SMT ROHS" (at 114.3 36.83 90)
+      (effects (font (size 1.27 1.27)) hide)
+    )
+    (pin "1")
+    (pin "2")
+    (instances
+      (project "Xing Signals XIAO"
+        (path "/1e761e62-995e-4cf3-b10a-8e152dd71096"
+          (reference "C3") (unit 1)
+        )
+      )
+    )
+  )
   (symbol (lib_id "Device:LED") (at 208.28 48.26 90) (unit 1)
     (in_bom yes) (on_board yes) (dnp no) (fields_autoplaced)
@@
       (effects (font (size 1.27 1.27)) (justify left))
     )
-    (property "Value" "+12V" (at 158.75 35.56 90)
+    (property "Value" "VIN" (at 158.75 35.56 90)
       (effects (font (size 1.27 1.27)) (justify left) hide)
     )

Commit message: Version 1.2
* Fixed a clearance issue between J3 and C2
* Moved D6 and D7 a bit closer to J3
Parts:
- C1, J1, J10, J3, J4, J6, J8, J9: now left out of the parts list
Changed lines of the file:
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@@
   )
   (symbol (lib_id "Device:C_Polarized_US") (at 224.79 34.29 0) (unit 1)
-    (in_bom yes) (on_board yes) (dnp no)
+    (in_bom no) (on_board yes) (dnp no)
     (property "Reference" "C1" (at 219.71 33.02 0)
       (effects (font (size 1.27 1.27)) (justify left))
@@
   )
   (symbol (lib_id "Connector:Conn_01x03_Pin") (at 254 107.95 90) (unit 1)
-    (in_bom yes) (on_board yes) (dnp no)
+    (in_bom no) (on_board yes) (dnp no)
     (property "Reference" "J10" (at 254 110.49 90)
       (effects (font (size 1.27 1.27)))
@@
   )
   (symbol (lib_id "Connector:Screw_Terminal_01x04") (at 17.78 140.97 180) (unit 1)
-    (in_bom yes) (on_board yes) (dnp no)
+    (in_bom no) (on_board yes) (dnp no)
     (property "Reference" "J8" (at 17.78 133.35 0)
       (effects (font (size 1.27 1.27)))
@@
   )
   (symbol (lib_id "Connector:Conn_01x03_Pin") (at 173.99 140.97 90) (unit 1)
-    (in_bom yes) (on_board yes) (dnp no) (fields_autoplaced)
+    (in_bom no) (on_board yes) (dnp no) (fields_autoplaced)
     (property "Reference" "J3" (at 173.99 143.51 90)
       (effects (font (size 1.27 1.27)))
@@
   )
   (symbol (lib_id "Connector:Conn_01x07_Pin") (at 76.2 53.34 180) (unit 1)
-    (in_bom yes) (on_board yes) (dnp no) (fields_autoplaced)
+    (in_bom no) (on_board yes) (dnp no) (fields_autoplaced)
     (property "Reference" "J9" (at 77.47 52.705 0)
       (effects (font (size 1.27 1.27)) (justify right))
@@
   )
   (symbol (lib_id "Connector_Generic:Conn_02x03_Top_Bottom") (at 245.11 139.7 90) (unit 1)
-    (in_bom yes) (on_board yes) (dnp no) (fields_autoplaced)
+    (in_bom no) (on_board yes) (dnp no) (fields_autoplaced)
     (property "Reference" "J4" (at 250.19 137.16 90)
       (effects (font (size 1.27 1.27)) (justify right))
@@
   )
   (symbol (lib_id "Connector:Barrel_Jack_Switch") (at 148.59 44.45 0) (unit 1)
-    (in_bom yes) (on_board yes) (dnp no) (fields_autoplaced)
+    (in_bom no) (on_board yes) (dnp no) (fields_autoplaced)
     (property "Reference" "J1" (at 148.59 35.56 0)
       (effects (font (size 1.27 1.27)))
@@
   )
   (symbol (lib_id "Connector:Conn_01x07_Pin") (at 93.98 53.34 0) (unit 1)
-    (in_bom yes) (on_board yes) (dnp no)
+    (in_bom no) (on_board yes) (dnp no)
     (property "Reference" "J6" (at 94.615 41.91 0)
       (effects (font (size 1.27 1.27)))
